Commit message: STL Mesh works

File: src/rover_description/urdf/bases/body.urdf.xacro (robot description, xacro)
@@ -11,6 +11,6 @@
                 <origin rpy="0 0 0" xyz="0 0 0" />
                 <geometry>
-                    <!-- <mesh filename="package://rover_description/meshes/bases/body_box2.stl" /> -->
-                    <box size="${body_box_length} ${body_box_width} ${body_box_depth}"/>
+                    <mesh filename="file://$(find rover_description)/meshes/bases/body_box.stl" />
+                 <!-- <box size="${body_box_length} ${body_box_width} ${body_box_depth}"/> -->
                 </geometry>
                 <material name="white" />

Commit message: First working innspace rover rovcer_description

File: src/rover_description/urdf/bases/body.urdf.xacro (robot description, xacro)
@@ -11,6 +11,6 @@
                 <origin rpy="0 0 0" xyz="0 0 0" />
                 <geometry>
-                    <!-- <mesh filename="package://rover_description/meshes/bases/body_box2.stl" /> -->
-                    <box size="${body_box_length} ${body_box_width} ${body_box_depth}"/>
+                    <mesh filename="file://$(find rover_description)/meshes/bases/body_box2.stl" />
+                    <!-- <box size="${body_box_length} ${body_box_width} ${body_box_depth}"/> -->
                 </geometry>
                 <material name="white" />
