Commit message: Description update and package xml depedencies added

File: src/rover_description/urdf/bases/rover_description.urdf.xacro (robot description, xacro)
@@ -47,5 +47,5 @@
   </link>
   <gazebo reference="chassis_link">
-        <material>Gazebo/Orange</material>
+        <material>Gazebo/White</material>
   </gazebo>
   <joint name="chassis_joint" type="fixed">
