Commit message: Readme installation note

File: src/rover_description/robots/rover_description.urdf.xacro (robot description, xacro)
@@ -45,4 +45,7 @@
     </collision>
   </link>
+  <gazebo reference="base_link">
+        <material>Gazebo/Orange</material>
+  </gazebo>
   <link
     name="front_right_wheel_link">
@@ -85,4 +88,7 @@
     </collision>
   </link>
+  <gazebo reference="front_right_wheel_link">
+        <material>Gazebo/Gray</material>
+  </gazebo>
   <joint
     name="front_right_wheel_joint"
