Commit message: Mesh added robot desrciption

File: src/rover_description/robots/rover.urdf.xacro (robot description, xacro)
@@ -1,7 +1,8 @@
 <?xml version="1.0"?>
-<robot xmlns:xacro="http://www.ros.org/wiki/xacro"  name="robot">
+<robot xmlns:xacro="http://www.ros.org/wiki/xacro"  name="rover">
     <!-- Include macros -->
     <xacro:include filename="$(find rover_description)/urdf/materials.xacro"/>
     <xacro:include filename="$(find rover_description)/urdf/inertials.xacro"/>
+    <xacro:include filename="$(find rover_description)/urdf/bases/body.urdf.xacro" />
     <!-- Example link -->
     <link name="base_link">
@@ -14,3 +15,8 @@
         </visual>
     </link>
+    <gazebo reference="base_link">
+        <material>Gazebo/Orange</material>
+    </gazebo>
+   <!-- body -->
+    <xacro:body parent="base_link" />
 </robot>

Commit message: Robot description moved to urdf/bases

File: src/rover_description/robots/rover.urdf.xacro (robot description, xacro)
@@ -4,19 +4,4 @@
     <xacro:include filename="$(find rover_description)/urdf/materials.xacro"/>
     <xacro:include filename="$(find rover_description)/urdf/inertials.xacro"/>
-    <xacro:include filename="$(find rover_description)/urdf/bases/body.urdf.xacro" />
-    <!-- Example link -->
-    <link name="base_link">
-        <visual>
-            <origin rpy="0 0 0" xyz="0 0 0" />
-            <geometry>
-                <box size="0.01 0.01 0.01"/>
-            </geometry>
-            <material name="orange" />
-        </visual>
-    </link>
-    <gazebo reference="base_link">
-        <material>Gazebo/Orange</material>
-    </gazebo>
-   <!-- body -->
-    <xacro:body parent="base_link" />
+    <xacro:include filename="$(find rover_description)/urdf/bases/rover_description.urdf.xacro" />
 </robot>

File: src/rover_description/urdf/bases/rover_description.urdf.xacro (robot description, xacro)
@@ -7,4 +7,6 @@
   <link
     name="base_link">
+  </link>
+  <link name="chassis_link">
     <inertial>
       <origin
@@ -27,5 +29,5 @@
       <geometry>
         <mesh
-          filename="file://$(find rover_description)/meshes/base_link.STL" />
+          filename="file://$(find rover_description)/meshes/chassis_link.STL" />
       </geometry>
       <material
@@ -41,11 +43,16 @@
       <geometry>
         <mesh
-          filename="file://$(find rover_description)/meshes/base_link.STL" />
-      </geometry>
-    </collision>
-  </link>
-  <gazebo reference="base_link">
+          filename="file://$(find rover_description)/meshes/chassis_link.STL" />
+      </geometry>
+    </collision>
+  </link>
+  <gazebo reference="chassis_link">
         <material>Gazebo/Orange</material>
   </gazebo>
+  <joint name="chassis_joint" type="fixed">
+    <parent link="base_link" />
+    <child link="chassis_link" />
+    <origin xyz="0 0 0" />
+  </joint>
   <link
     name="front_right_wheel_link">
@@ -55,5 +62,5 @@
         rpy="0 0 0" />
       <mass
-        value="7" />
+        value="1" />
       <inertia
         ixx="0.440773403043026"
@@ -111,5 +118,5 @@
         rpy="0 0 0" />
       <mass
-        value="7" />
+        value="1" />
       <inertia
         ixx="0.440773403043026"
@@ -144,4 +151,7 @@
     </collision>
   </link>
+  <gazebo reference="rear_right_wheel_link">
+        <material>Gazebo/Gray</material>
+  </gazebo>
   <joint
     name="rear_right_wheel_joint"
@@ -164,5 +174,5 @@
         rpy="0 0 0" />
       <mass
-        value="7" />
+        value="1" />
       <inertia
         ixx="0.440773403043026"
@@ -197,4 +207,7 @@
     </collision>
   </link>
+  <gazebo reference="front_left_wheel_link">
+        <material>Gazebo/Gray</material>
+  </gazebo>
   <joint
     name="front_left_wheel_joint"
@@ -217,5 +230,5 @@
         rpy="0 0 0" />
       <mass
-        value="7" />
+        value="1" />
       <inertia
         ixx="0.440773403043026"
@@ -250,4 +263,7 @@
     </collision>
   </link>
+  <gazebo reference="rear_left_wheel_link">
+        <material>Gazebo/Gray</material>
+  </gazebo>
   <joint
     name="rear_left_wheel_joint"

Commit message: Oak_D sensor added to siulation from macro

File: src/rover_description/robots/rover.urdf.xacro (robot description, xacro)
@@ -4,4 +4,4 @@
     <xacro:include filename="$(find rover_description)/urdf/materials.xacro"/>
     <xacro:include filename="$(find rover_description)/urdf/bases/rover_description.urdf.xacro" />
-    <xacro:include filename="$(find rover_description)/urdf/sensors/camera.urdf.xacro" />
+    <xacro:include filename="$(find rover_description)/urdf/sensors/camera_2.urdf.xacro" />
 </robot>

File: src/rover_description/urdf/sensors/camera.urdf.xacro (robot description, xacro)
@@ -34,8 +34,9 @@
     <joint name="camera_optical_joint" type="fixed">
       <parent link="camera_link" />
-      <child link="camera_link_optical" />
+      <child link="camera_rgb_link_optical camera_stereo_link_optical" />
       <origin xyz="0 0 0" rpy="${-pi/2} 0 ${-pi/2}"/>
     </joint>
-    <link name="camera_link_optical"></link>
+    <link name="camera_rgb_link_optical"></link>
+    <link name="camera_stereo_link_optical"></link>
     <gazebo reference="camera_link">
       <material>Gazebo/DarkGrey</material>
@@ -87,3 +88,61 @@
     </sensor>
     </gazebo>
+    <gazebo reference="camera_link">
+      <material>Gazebo/DarkGrey</material>
+      <sensor type="multicamera" name="stereo_camera">
+        <update_rate>30.0</update_rate>
+        <camera name="left">
+          <horizontal_fov>1.2566</horizontal_fov>
+          <image>
+            <width>1200</width>
+            <height>800</height>
+      <format>L8</format>
+      <!--   <format>R8G8B8</format> -->
+          </image>
+          <clip>
+            <near>0.3</near>
+            <far>35</far>
+          </clip>
+          <noise>
+            <type>gaussian</type>
+            <mean>0.0</mean>
+            <stddev>0.007</stddev>
+          </noise>
+        </camera>
+        <camera name="right">
+          <pose>0 -0.07 0 0 0 0</pose>
+          <horizontal_fov>1.1.2566</horizontal_fov>
+          <image>
+            <width>1200</width>
+            <height>800</height>
+      <format>L8</format>
+      <!--   <format>R8G8B8</format> -->
+          </image>
+          <clip>
+            <near>0.3</near>
+            <far>35</far>
+          </clip>
+          <noise>
+            <type>gaussian</type>
+            <mean>0.0</mean>
+            <stddev>0.007</stddev>
+          </noise>
+        </camera>
+        <plugin name="stereo_camera_controller" filename="libgazebo_ros_multicamera.so">
+          <alwaysOn>true</alwaysOn>
+          <updateRate>0.0</updateRate>
+    <cameraName>oakd_${mount_point}/camera</cameraName>
+          <imageTopicName>image_raw</imageTopicName>
+          <cameraInfoTopicName>camera_info</cameraInfoTopicName>
+    <frameName>camera_optical_frame</frameName>
+          <!--<rightFrameName>right_camera_optical_frame</rightFrameName>-->
+          <hackBaseline>0.075</hackBaseline>
+          <distortionK1>0.0</distortionK1>
+          <distortionK2>0.0</distortionK2>
+          <distortionK3>0.0</distortionK3>
+          <distortionT1>0.0</distortionT1>
+          <distortionT2>0.0</distortionT2>
+        </plugin>
+      </sensor>
+  </gazebo>
 </robot>

File: src/rover_description/urdf/sensors/oak_d.xacro (robot description, xacro)
@@ -3,178 +3,179 @@
 <robot name="oakd" xmlns:xacro="http://ros.org/wiki/xacro">
       <xacro:macro name="oakd_link" params="mount_point">
-      <xacro:property name="oakd_length" value="0.0803" />
-      <xacro:property name="oakd_width" value="0.0957" />
-      <xacro:property name="oakd_depth" value="0.1267" />
-      <xacro:property name="oakd_mass" value="0.15" />
-      <link name="oakd_${mount_point}">
-             <pose>0.0 0.0 0.0 0.0 0.0 0.0</pose>
-          <visual>
-              <origin rpy="0 0 0" xyz="0 0 0" />
-              <geometry>
-                      <mesh filename="package://oakd_description/meshes/sensors/OAK-D.dae" />
-              </geometry>
-               <material name="black" />
-          </visual>
-          <collision>
-              <origin rpy="0 0 0" xyz="0 0 0" />
-              <geometry>
-                  <box size="${oakd_length} ${oakd_width} ${oakd_depth}"/>
-              </geometry>
-          </collision>
-          <xacro:solid_cuboid_inertial
-              rpy="0 0 0" xyz="0 0 0"
-              mass="${oakd_mass}"
-              x="${oakd_length}" y="${oakd_width}" z="${oakd_depth}" />
-      </link>
-      <!-- Add dummy joint for camera_optical_frame to link back to base_link -->
-      <joint name="camera_optical_joint" type="fixed">
-      <!-- Point cloud frustrum is 90 degrees off from visual frame -->
-           <origin rpy="-1.57079632769 0 -1.570796332769" xyz="0 0 0" />
-	   <parent link="oakd_${mount_point}" />
-	   <child link="camera_optical_frame" />
-	</joint>
-	<!-- Add dummy link for camera_optical_frame to link back to base_link -->
-        <link name="camera_optical_frame">
-        <inertial>
-	  <mass value="0.001" />
-	  <origin xyz="0 0 0" />
-	  <inertia ixx="0.0001" ixy="0.0" ixz="0.0" iyy="0.0001" iyz="0.0" izz="0.0001" />
-          </inertial>
-  </link>
-  <!-- Dummy joints for rgb camera to link back to base_link -->
-        <joint name="camera_rgb_optical_joint" type="fixed">
-           <origin rpy="0 0 0" xyz="0 0 0" />
-	   <parent link="oakd_${mount_point}" />
-	   <child link="camera_rgb_optical_frame" />
-	</joint>
-	<!-- Add dummy link for camera_optical_frame to link back to base_link -->
-        <link name="camera_rgb_optical_frame">
-        <inertial>
-	  <mass value="0.001" />
-	  <origin xyz="0 0 0" />
-	  <inertia ixx="0.0001" ixy="0.0" ixz="0.0" iyy="0.0001" iyz="0.0" izz="0.0001" />
-          </inertial>
-  </link>
-  <!-- Gazebo plugin for greyscale left/right stereo pairs -->
-      <gazebo reference="oakd_${mount_point}">
-    <material>Gazebo/DarkGrey</material>
-    <sensor type="multicamera" name="stereo_camera">
-      <update_rate>30.0</update_rate>
-      <camera name="left">
-        <horizontal_fov>1.2566</horizontal_fov>
-        <image>
-          <width>1200</width>
-          <height>800</height>
-	  <format>L8</format>
-	  <!--   <format>R8G8B8</format> -->
-        </image>
-        <clip>
-          <near>0.3</near>
-          <far>35</far>
-        </clip>
-        <noise>
-          <type>gaussian</type>
-          <mean>0.0</mean>
-          <stddev>0.007</stddev>
-        </noise>
-      </camera>
-      <camera name="right">
-        <pose>0 -0.07 0 0 0 0</pose>
-        <horizontal_fov>1.1.2566</horizontal_fov>
-        <image>
-          <width>1200</width>
-          <height>800</height>
-	  <format>L8</format>
-	  <!--   <format>R8G8B8</format> -->
-        </image>
-        <clip>
-          <near>0.3</near>
-          <far>35</far>
-        </clip>
-        <noise>
-          <type>gaussian</type>
-          <mean>0.0</mean>
-          <stddev>0.007</stddev>
-        </noise>
-      </camera>
-      <plugin name="stereo_camera_controller" filename="libgazebo_ros_multicamera.so">
-        <alwaysOn>true</alwaysOn>
-        <updateRate>0.0</updateRate>
-	<cameraName>oakd_${mount_point}/camera</cameraName>
-        <imageTopicName>image_raw</imageTopicName>
-        <cameraInfoTopicName>camera_info</cameraInfoTopicName>
-	<frameName>camera_optical_frame</frameName>
-        <!--<rightFrameName>right_camera_optical_frame</rightFrameName>-->
-        <hackBaseline>0.075</hackBaseline>
-        <distortionK1>0.0</distortionK1>
-        <distortionK2>0.0</distortionK2>
-        <distortionK3>0.0</distortionK3>
-        <distortionT1>0.0</distortionT1>
-        <distortionT2>0.0</distortionT2>
-      </plugin>
-    </sensor>
-  </gazebo>
- <!-- Gazebo plugin for center RGB camera -->
-   <gazebo reference="oakd_${mount_point}">
-      <material>Gazebo/White</material>
-      <sensor type="camera" name="oakd_rgb_${mount_point}">
-      <update_rate>30.0</update_rate>
-      <camera name="head">
-        <horizontal_fov>1.3962634</horizontal_fov>
-        <image>
-          <width>800</width>
-          <height>800</height>
-          <format>R8G8B8</format>
-        </image>
-        <clip>
-          <near>0.02</near>
-          <far>300</far>
-        </clip>
-        <noise>
-          <type>gaussian</type>
-          <!-- Noise is sampled independently per pixel on each frame.
-               That pixel's noise value is added to each of its color
-               channels, which at that point lie in the range [0,1]. -->
-          <mean>0.0</mean>
-          <stddev>0.007</stddev>
-        </noise>
-      </camera>
-      <plugin name="camera_controller" filename="libgazebo_ros_camera.so">
-        <alwaysOn>true</alwaysOn>
-        <updateRate>0.0</updateRate>
-        <cameraName>oakd_rgb_${mount_point}</cameraName>
-        <imageTopicName>image_raw</imageTopicName>
-        <cameraInfoTopicName>camera_info</cameraInfoTopicName>
-        <frameName>camera_rgb_link_optical</frameName>
-        <!-- setting hackBaseline to anything but 0.0 will cause a misalignment
-            between the gazebo sensor image and the frame it is supposed to
-            be attached to -->
-        <hackBaseline>0.0</hackBaseline>
-        <distortionK1>0.0</distortionK1>
-        <distortionK2>0.0</distortionK2>
-        <distortionK3>0.0</distortionK3>
-        <distortionT1>0.0</distortionT1>
-        <distortionT2>0.0</distortionT2>
-        <CxPrime>0</CxPrime>
-        <Cx>0.0</Cx>
-        <Cy>0.0</Cy>
-        <focalLength>0.0</focalLength>
-      </plugin>
-    </sensor>
-  </gazebo>
-      <gazebo reference="oakd_joint_${mount_point}">
-          <!-- <disableFixedJointLumping>true</disableFixedJointLumping>  -->
-          <!-- <preserveFixedJoint>true</preserveFixedJoint> -->
-      </gazebo>
-    </xacro:macro>
-    <xacro:macro name="oakd_joint" params="x y z roll pitch yaw mount_point" >
-        <joint name="oakd_joint_${mount_point}" type="fixed">
-                <origin rpy="${roll} ${pitch} ${yaw}" xyz="${x}+0.1 ${y}-0.01 ${z}"/>
-            <parent link="base_link" />
-            <child link="oakd_${mount_point}" />
-        </joint>
+        <xacro:property name="oakd_length" value="0.0803" />
+        <xacro:property name="oakd_width" value="0.0957" />
+        <xacro:property name="oakd_depth" value="0.1267" />
+        <xacro:property name="oakd_mass" value="0.15" />
+        <link name="oakd_${mount_point}">
+              <pose>0.0 0.0 0.0 0.0 0.0 0.0</pose>
+            <visual>
+                <origin rpy="0 0 0" xyz="0 0 0" />
+                <geometry>
+                        <mesh filename="file://$(find rover_description)/meshes/sensors/OAK-D.dae" />
+                </geometry>
+                <material name="black" />
+            </visual>
+            <collision>
+                <origin rpy="0 0 0" xyz="0 0 0" />
+                <geometry>
+                    <box size="${oakd_length} ${oakd_width} ${oakd_depth}"/>
+                </geometry>
+            </collision>
+            <xacro:solid_cuboid_inertial
+                rpy="0 0 0" xyz="0 0 0"
+                mass="${oakd_mass}"
+                x="${oakd_length}" y="${oakd_width}" z="${oakd_depth}" />
+        </link>
+        <!-- Add dummy joint for camera_optical_frame to link back to base_link -->
+        <joint name="camera_optical_joint" type="fixed">
+        <!-- Point cloud frustrum is 90 degrees off from visual frame -->
+            <origin rpy="-1.57079632769 0 -1.570796332769" xyz="0 0 0" />
+      <parent link="oakd_${mount_point}" />
+      <child link="camera_optical_frame" />
+    </joint>
+    <!-- Add dummy link for camera_optical_frame to link back to base_link -->
+          <link name="camera_optical_frame">
+          <inertial>
+      <mass value="0.001" />
+      <origin xyz="0 0 0" />
+      <inertia ixx="0.0001" ixy="0.0" ixz="0.0" iyy="0.0001" iyz="0.0" izz="0.0001" />
+            </inertial>
+    </link>
+    <!-- Dummy joints for rgb camera to link back to base_link -->
+          <joint name="camera_rgb_optical_joint" type="fixed">
+            <origin rpy="0 0 0" xyz="0 0 0" />
+      <parent link="oakd_${mount_point}" />
+      <child link="camera_rgb_optical_frame" />
+    </joint>
+    <!-- Add dummy link for camera_optical_frame to link back to base_link -->
+          <link name="camera_rgb_optical_frame">
+          <inertial>
+      <mass value="0.001" />
+      <origin xyz="0 0 0" />
+      <inertia ixx="0.0001" ixy="0.0" ixz="0.0" iyy="0.0001" iyz="0.0" izz="0.0001" />
+            </inertial>
+    </link>
+    <!-- Gazebo plugin for greyscale left/right stereo pairs -->
+        <gazebo reference="oakd_${mount_point}">
+      <material>Gazebo/DarkGrey</material>
+      <sensor type="multicamera" name="stereo_camera">
+        <update_rate>30.0</update_rate>
+        <camera name="left">
+          <horizontal_fov>1.2566</horizontal_fov>
+          <image>
+            <width>1200</width>
+            <height>800</height>
+      <format>L8</format>
+      <!--   <format>R8G8B8</format> -->
+          </image>
+          <clip>
+            <near>0.3</near>
+            <far>35</far>
+          </clip>
+          <noise>
+            <type>gaussian</type>
+            <mean>0.0</mean>
+            <stddev>0.007</stddev>
+          </noise>
+        </camera>
+        <camera name="right">
+          <pose>0 -0.07 0 0 0 0</pose>
+          <horizontal_fov>1.1.2566</horizontal_fov>
+          <image>
+            <width>1200</width>
+            <height>800</height>
+      <format>L8</format>
+      <!--   <format>R8G8B8</format> -->
+          </image>
+          <clip>
+            <near>0.3</near>
+            <far>35</far>
+          </clip>
+          <noise>
+            <type>gaussian</type>
+            <mean>0.0</mean>
+            <stddev>0.007</stddev>
+          </noise>
+        </camera>
+        <plugin name="stereo_camera_controller" filename="libgazebo_ros_multicamera.so">
+          <alwaysOn>true</alwaysOn>
+          <updateRate>0.0</updateRate>
+    <cameraName>oakd_${mount_point}/camera</cameraName>
+          <imageTopicName>image_raw</imageTopicName>
+          <cameraInfoTopicName>camera_info</cameraInfoTopicName>
+    <frameName>camera_optical_frame</frameName>
+          <!--<rightFrameName>right_camera_optical_frame</rightFrameName>-->
+          <hackBaseline>0.075</hackBaseline>
+          <distortionK1>0.0</distortionK1>
+          <distortionK2>0.0</distortionK2>
+          <distortionK3>0.0</distortionK3>
+          <distortionT1>0.0</distortionT1>
+          <distortionT2>0.0</distortionT2>
+        </plugin>
+      </sensor>
+    </gazebo>
+  <!-- Gazebo plugin for center RGB camera -->
+    <gazebo reference="oakd_${mount_point}">
+        <!-- <material>Gazebo/White</material> -->
+        <sensor type="camera" name="oakd_rgb_${mount_point}">
+        <visualize>true</visualize>
+        <update_rate>30.0</update_rate>
+        <camera name="head">
+          <horizontal_fov>1.3962634</horizontal_fov>
+          <image>
+            <width>800</width>
+            <height>800</height>
+            <format>R8G8B8</format>
+          </image>
+          <clip>
+            <near>0.02</near>
+            <far>300</far>
+          </clip>
+          <noise>
+            <type>gaussian</type>
+            <!-- Noise is sampled independently per pixel on each frame.
+                That pixel's noise value is added to each of its color
+                channels, which at that point lie in the range [0,1]. -->
+            <mean>0.0</mean>
+            <stddev>0.007</stddev>
+          </noise>
+        </camera>
+        <plugin name="camera_controller" filename="libgazebo_ros_camera.so">
+          <alwaysOn>true</alwaysOn>
+          <updateRate>0.0</updateRate>
+          <cameraName>oakd_rgb_${mount_point}</cameraName>
+          <imageTopicName>image_raw</imageTopicName>
+          <cameraInfoTopicName>camera_info</cameraInfoTopicName>
+          <frameName>camera_rgb_link_optical</frameName>
+          <!-- setting hackBaseline to anything but 0.0 will cause a misalignment
+              between the gazebo sensor image and the frame it is supposed to
+              be attached to -->
+          <hackBaseline>0.0</hackBaseline>
+          <distortionK1>0.0</distortionK1>
+          <distortionK2>0.0</distortionK2>
+          <distortionK3>0.0</distortionK3>
+          <distortionT1>0.0</distortionT1>
+          <distortionT2>0.0</distortionT2>
+          <CxPrime>0</CxPrime>
+          <Cx>0.0</Cx>
+          <Cy>0.0</Cy>
+          <focalLength>0.0</focalLength>
+        </plugin>
+      </sensor>
+    </gazebo>
         <gazebo reference="oakd_joint_${mount_point}">
-            <preserveFixedJoint>true</preserveFixedJoint>
+            <!-- <disableFixedJointLumping>true</disableFixedJointLumping>  -->
+            <!-- <preserveFixedJoint>true</preserveFixedJoint> -->
         </gazebo>
+      </xacro:macro>
+      <xacro:macro name="oakd_joint" params="x y z roll pitch yaw mount_point" >
+          <joint name="oakd_joint_${mount_point}" type="fixed">
+                  <origin rpy="${roll} ${pitch} ${yaw}" xyz="${x}+0.1 ${y}-0.01 ${z}"/>
+              <parent link="base_link" />
+              <child link="oakd_${mount_point}" />
+          </joint>
+          <gazebo reference="oakd_joint_${mount_point}">
+              <preserveFixedJoint>true</preserveFixedJoint>
+          </gazebo>
     </xacro:macro>
 </robot>
