Commit message: Depth camera simulation

File: src/rover_description/robots/rover.urdf.xacro (robot description, xacro)
@@ -4,4 +4,4 @@
     <xacro:include filename="$(find rover_description)/urdf/materials.xacro"/>
     <xacro:include filename="$(find rover_description)/urdf/bases/rover_description.urdf.xacro" />
-    <xacro:include filename="$(find rover_description)/urdf/sensors/camera_2.urdf.xacro" />
+    <xacro:include filename="$(find rover_description)/urdf/sensors/camera.urdf.xacro" />
 </robot>

File: src/rover_description/urdf/sensors/camera.urdf.xacro (robot description, xacro)
@@ -3,146 +3,10 @@
 <robot xmlns:xacro="http://ros.org/wiki/xacro" name="camera">
     <xacro:include filename="$(find rover_description)/urdf/inertials.xacro"/>
-    <xacro:property name="oakd_length" value="0.0803" />
-    <xacro:property name="oakd_width" value="0.0957" />
-    <xacro:property name="oakd_depth" value="0.1267" />
-    <xacro:property name="oakd_mass" value="0.15" />
-    <joint name="camera_joint" type="fixed">
+    <xacro:include filename="$(find rover_description)/urdf/sensors/oak_d.xacro"/>
+    <joint name="oakd_joint" type="fixed">
       <parent link="chassis_link" />
-      <child link="camera_link" />
+      <child link="oakd_front" />
       <origin xyz="0.44 0 0.07" rpy="0 0 0"/>
     </joint>
-    <link name="camera_link">
-      <pose> 0 0 0 0 0 0 </pose>
-      <visual>
-          <geometry>
-            <mesh filename="file://$(find rover_description)/meshes/sensors/OAK-D.dae" />
-            <!-- <box size="0.010 0.03 0.03"/> -->
-          </geometry>
-          <material name="black" />
-      </visual>
-      <collision>
-          <origin rpy="0 0 0" xyz="0 0 0" />
-          <geometry>
-              <box size="${oakd_length} ${oakd_width} ${oakd_depth}"/>
-          </geometry>
-      </collision>
-      <xacro:solid_cuboid_inertial
-              rpy="0 0 0" xyz="0 0 0"
-              mass="${oakd_mass}"
-              x="${oakd_length}" y="${oakd_width}" z="${oakd_depth}" />
-    </link>
-    <joint name="camera_optical_joint" type="fixed">
-      <parent link="camera_link" />
-      <child link="camera_rgb_link_optical camera_stereo_link_optical" />
-      <origin xyz="0 0 0" rpy="${-pi/2} 0 ${-pi/2}"/>
-    </joint>
-    <link name="camera_rgb_link_optical"></link>
-    <link name="camera_stereo_link_optical"></link>
-    <gazebo reference="camera_link">
-      <material>Gazebo/DarkGrey</material>
-      <sensor type="camera" name="camera">
-        <pose> 0 0 0 0 0 0 </pose>
-        <visualize>true</visualize>
-        <update_rate>30.0</update_rate>
-        <camera name="head">
-          <horizontal_fov>1.3962634</horizontal_fov>
-          <image>
-            <width>800</width>
-            <height>800</height>
-            <format>R8G8B8</format>
-          </image>
-          <clip>
-            <near>0.02</near>
-            <far>300</far>
-          </clip>
-          <noise>
-            <type>gaussian</type>
-            <!-- Noise is sampled independently per pixel on each frame.
-                That pixel's noise value is added to each of its color
-                channels, which at that point lie in the range [0,1]. -->
-            <mean>0.0</mean>
-            <stddev>0.007</stddev>
-          </noise>
-        </camera>
-        <plugin name="camera_controller" filename="libgazebo_ros_camera.so">
-          <alwaysOn>true</alwaysOn>
-          <updateRate>0.0</updateRate>
-          <cameraName>camera_rgb</cameraName>
-          <imageTopicName>image_raw</imageTopicName>
-          <cameraInfoTopicName>camera_info</cameraInfoTopicName>
-          <frameName>camera_rgb_link_optical</frameName>
-          <!-- setting hackBaseline to anything but 0.0 will cause a misalignment
-              between the gazebo sensor image and the frame it is supposed to
-              be attached to -->
-          <hackBaseline>0.0</hackBaseline>
-          <distortionK1>0.0</distortionK1>
-          <distortionK2>0.0</distortionK2>
-          <distortionK3>0.0</distortionK3>
-          <distortionT1>0.0</distortionT1>
-          <distortionT2>0.0</distortionT2>
-          <CxPrime>0</CxPrime>
-          <Cx>0.0</Cx>
-          <Cy>0.0</Cy>
-          <focalLength>0.0</focalLength>
-        </plugin>
-    </sensor>
-    </gazebo>
-    <gazebo reference="camera_link">
-      <material>Gazebo/DarkGrey</material>
-      <sensor type="multicamera" name="stereo_camera">
-        <update_rate>30.0</update_rate>
-        <camera name="left">
-          <horizontal_fov>1.2566</horizontal_fov>
-          <image>
-            <width>1200</width>
-            <height>800</height>
-      <format>L8</format>
-      <!--   <format>R8G8B8</format> -->
-          </image>
-          <clip>
-            <near>0.3</near>
-            <far>35</far>
-          </clip>
-          <noise>
-            <type>gaussian</type>
-            <mean>0.0</mean>
-            <stddev>0.007</stddev>
-          </noise>
-        </camera>
-        <camera name="right">
-          <pose>0 -0.07 0 0 0 0</pose>
-          <horizontal_fov>1.1.2566</horizontal_fov>
-          <image>
-            <width>1200</width>
-            <height>800</height>
-      <format>L8</format>
-      <!--   <format>R8G8B8</format> -->
-          </image>
-          <clip>
-            <near>0.3</near>
-            <far>35</far>
-          </clip>
-          <noise>
-            <type>gaussian</type>
-            <mean>0.0</mean>
-            <stddev>0.007</stddev>
-          </noise>
-        </camera>
-        <plugin name="stereo_camera_controller" filename="libgazebo_ros_multicamera.so">
-          <alwaysOn>true</alwaysOn>
-          <updateRate>0.0</updateRate>
-    <cameraName>oakd_${mount_point}/camera</cameraName>
-          <imageTopicName>image_raw</imageTopicName>
-          <cameraInfoTopicName>camera_info</cameraInfoTopicName>
-    <frameName>camera_optical_frame</frameName>
-          <!--<rightFrameName>right_camera_optical_frame</rightFrameName>-->
-          <hackBaseline>0.075</hackBaseline>
-          <distortionK1>0.0</distortionK1>
-          <distortionK2>0.0</distortionK2>
-          <distortionK3>0.0</distortionK3>
-          <distortionT1>0.0</distortionT1>
-          <distortionT2>0.0</distortionT2>
-        </plugin>
-      </sensor>
-  </gazebo>
+    <xacro:oakd_link mount_point="front"/>
 </robot>

File: src/rover_description/urdf/sensors/oak_d.xacro (robot description, xacro)
@@ -57,7 +57,7 @@
     </link>
     <!-- Gazebo plugin for greyscale left/right stereo pairs -->
-        <gazebo reference="oakd_${mount_point}">
+    <gazebo reference="oakd_${mount_point}">
       <material>Gazebo/DarkGrey</material>
-      <sensor type="multicamera" name="stereo_camera">
+      <sensor type="multicamera" name="oakd_stereo_${mount_point}">
         <update_rate>30.0</update_rate>
         <camera name="left">
@@ -98,5 +98,6 @@
           </noise>
         </camera>
-        <plugin name="stereo_camera_controller" filename="libgazebo_ros_multicamera.so">
+        <plugin name="stereo_camera_controller" filename="libgazebo_ros_camera.so">
+        <!-- libgazebo_ros_multicamera.so -->
           <alwaysOn>true</alwaysOn>
           <updateRate>0.0</updateRate>
@@ -115,4 +116,28 @@
       </sensor>
     </gazebo>
+  <gazebo reference="oakd_${mount_point}">
+    <sensor name="oakd_depth_${mount_point}" type="depth">
+      <visualize>true</visualize>
+      <update_rate>10</update_rate>
+      <camera>
+          <horizontal_fov>1.2566</horizontal_fov>
+          <image>
+            <width>1200</width>
+            <height>800</height>
+            <format>B8G8R8</format>
+      <!--   <format>R8G8B8</format> -->
+          </image>
+          <clip>
+            <near>0.05</near>
+            <far>8.0</far>
+          </clip>
+      </camera>
+      <plugin name="depth_camera_controller" filename="libgazebo_ros_camera.so">
+        <frame_name>camera_optical_frame</frame_name>
+        <min_depth>0.1</min_depth>
+        <max_depth>100.0</max_depth>
+      </plugin>
+    </sensor>
+  </gazebo>
   <!-- Gazebo plugin for center RGB camera -->
     <gazebo reference="oakd_${mount_point}">
