Commit message: SLAM is drifting but works and added maze world

File: src/rover_description/urdf/sensors/lidar.urdf.xacro (robot description, xacro)
@@ -23,5 +23,5 @@
     <parent link="chassis_link"/>
     <child link="lidar_link"/>
-    <origin xyz="0.3 0 -0.1" rpy="0 0 0"/>
+    <origin xyz="0.35 0 -0.1" rpy="0 0 0"/>
     </joint>
     <gazebo reference="lidar_link">
@@ -42,5 +42,5 @@
         <range>
             <min>0.120000</min>
-            <max>3.5</max>
+            <max>10</max>
             <resolution>0.015000</resolution>
         </range>
